Commit message: .

File: 3D_CAD_Scara1/urdf/3D_CAD_Scara1.urdf (robot description, URDF)
Before this commit: robot 3D_CAD_Scara, 4 links, 3 joints
Links:
- removed link world
- added link End_effector, mass 3.121; collision mesh filename=package://3D_CAD_Scara1/meshes/End_effector.STL; visual mesh filename=package://3D_CAD_Scara1/meshes/End_effector.STL
- added link base_link, mass 7.81592864600267; collision mesh filename=package://3D_CAD_Scara1/meshes/base_link.STL; visual mesh filename=package://3D_CAD_Scara1/meshes/base_link.STL
- link Link02_Link: geometry collision mesh filename=package://3D_CAD_Scara1/meshes/Link02_Link.STL; visual mesh filename=package://3D_CAD_Scara1/meshes/Link02_Link.STL
- link Link03_Link: geometry collision mesh filename=package://3D_CAD_Scara1/meshes/Link03_Link.STL; visual mesh filename=package://3D_CAD_Scara1/meshes/Link03_Link.STL
- link Link1_Link: geometry collision mesh filename=package://3D_CAD_Scara1/meshes/Link1_Link.STL; visual mesh filename=package://3D_CAD_Scara1/meshes/Link1_Link.STL
Joints:
- added joint end_efector: type fixed, parent Link03_Link, child End_effector, origin xyz=0 0 -0.31 rpy=0 0 0, axis 0 0 0
- joint joint01_joint: origin xyz=0 0 0.22 rpy=0 0 -0.26199 -> xyz=0 0 0.22 rpy=0 0 -0.0076361; parent world -> base_link
- joint joint02_joint: origin xyz=0.55 0 0.1 rpy=0 0 -1.4556 -> xyz=0.55 0 0.1 rpy=0 0 -0.091166
- joint joint03_joint: origin xyz=0.55 0.050125 0 rpy=0 0 0 -> xyz=0.55 0.00012531 0.054965 rpy=0 0 0
