Commit message: 02

File: 3D_CAD_Scara/urdf/3D_CAD_Scara.urdf (robot description, URDF)
Before this commit: robot 3D_CAD_Scara1, 5 links, 4 joints
Links:
- removed link End_effector
- removed link Link1_Link
- added link End_efector_Link, mass 2.621; collision mesh filename=package://3D_CAD_Scara/meshes/End_efector_Link.STL; visual mesh filename=package://3D_CAD_Scara/meshes/End_efector_Link.STL
- added link Link01_Link, mass 6.88681009624485; collision mesh filename=package://3D_CAD_Scara/meshes/Link01_Link.STL; visual mesh filename=package://3D_CAD_Scara/meshes/Link01_Link.STL
- link Link02_Link: mass 6.45815878743564 -> 4.46317135032901; geometry collision mesh filename=package://3D_CAD_Scara/meshes/Link02_Link.STL; visual mesh filename=package://3D_CAD_Scara/meshes/Link02_Link.STL
- link Link03_Link: mass 3.121 -> 2.621; geometry collision mesh filename=package://3D_CAD_Scara/meshes/Link03_Link.STL; visual mesh filename=package://3D_CAD_Scara/meshes/Link03_Link.STL
- link base_link: mass 7.81592864600267 -> 6.24513231920778; geometry collision mesh filename=package://3D_CAD_Scara/meshes/base_link.STL; visual mesh filename=package://3D_CAD_Scara/meshes/base_link.STL
Joints:
- removed joint end_efector
- removed joint joint01_joint
- added joint Endefector_joint: type fixed, parent Link03_Link, child End_efector_Link, origin xyz=0 0 -0.26 rpy=0 0 0, axis 0 0 0
- added joint Joint01_joint: type continuous, parent base_link, child Link01_Link, origin xyz=0 0 0.17 rpy=0 0 0, axis 0 0 1
- joint joint02_joint: limit lower=0 upper=0 effort=0 velocity=0 -> (none); origin xyz=0.55 0 0.1 rpy=0 0 -0.091166 -> xyz=0.34999 -0.0025138 0.1 rpy=0 0 0; parent Link1_Link -> Link01_Link
- joint joint03_joint: limit lower=-0.0049658 upper=0.17503 effort=0 velocity=0 -> lower=0 upper=0.13 effort=0 velocity=0; origin xyz=0.55 0.00012531 0.054965 rpy=0 0 0 -> xyz=0.34988 0.0091808 0.05 rpy=0 0 0
