Commit message: .
Clean the my_robot folder

File: from_lab0_requirement/my_robot/robot.urdf (robot description, URDF)
Before this commit: robot 3D_CAD_Scara, 5 links, 4 joints
Links:
- link End_efector_Link: geometry collision mesh filename=package://my_robot/meshes/End_efector_Link.STL; visual mesh filename=package://my_robot/meshes/End_efector_Link.STL
- link Link01_Link: geometry collision mesh filename=package://my_robot/meshes/Link01_Link.STL; visual mesh filename=package://my_robot/meshes/Link01_Link.STL
- link Link02_Link: geometry collision mesh filename=package://my_robot/meshes/Link02_Link.STL; visual mesh filename=package://my_robot/meshes/Link02_Link.STL
- link Link03_Link: geometry collision mesh filename=package://my_robot/meshes/Link03_Link.STL; visual mesh filename=package://my_robot/meshes/Link03_Link.STL
- link base_link: geometry collision mesh filename=package://my_robot/meshes/base_link.STL; visual mesh filename=package://my_robot/meshes/base_link.STL
