Commit message: jj

File: 3D_CAD_Scara3/urdf/3D_CAD_Scara3.urdf (robot description, URDF)
Before this commit: robot 3D_CAD_Scara1, 5 links, 4 joints
Links:
- removed link End_effector
- removed link Link1_Link
- added link End_efector_Link, mass 2.621; collision mesh filename=package://3D_CAD_Scara3/meshes/End_efector_Link.STL; visual mesh filename=package://3D_CAD_Scara3/meshes/End_efector_Link.STL
- added link Link01_Link, mass 6.88681009624485; collision mesh filename=package://3D_CAD_Scara3/meshes/Link01_Link.STL; visual mesh filename=package://3D_CAD_Scara3/meshes/Link01_Link.STL
- link Link02_Link: mass 6.45815878743564 -> 4.46317135032902; geometry collision mesh filename=package://3D_CAD_Scara3/meshes/Link02_Link.STL; visual mesh filename=package://3D_CAD_Scara3/meshes/Link02_Link.STL
- link Link03_Link: mass 3.121 -> 2.621; geometry collision mesh filename=package://3D_CAD_Scara3/meshes/Link03_Link.STL; visual mesh filename=package://3D_CAD_Scara3/meshes/Link03_Link.STL
- link base_link: mass 7.81592864600267 -> 6.24513231920778; geometry collision mesh filename=package://3D_CAD_Scara3/meshes/base_link.STL; visual mesh filename=package://3D_CAD_Scara3/meshes/base_link.STL
Joints:
- removed joint end_efector
- removed joint joint01_joint
- added joint Endefector_joint: type fixed, parent Link03_Link, child End_efector_Link, origin xyz=0 0 0.03 rpy=0 0 1.8765, axis 0 0 0
- added joint Joint01_joint: type continuous, parent base_link, child Link01_Link, origin xyz=0 0 0.17 rpy=0 0 0, axis 0 0 1
- joint joint02_joint: limit lower=0 upper=0 effort=0 velocity=0 -> (none); origin xyz=0.55 0 0.1 rpy=0 0 -0.091166 -> xyz=-0.15026 0.3161 0.1 rpy=0 0 0; parent Link1_Link -> Link01_Link
- joint joint03_joint: limit lower=-0.0049658 upper=0.17503 effort=0 velocity=0 -> lower=0 upper=0.130 effort=0 velocity=0; origin xyz=0.55 0.00012531 0.054965 rpy=0 0 0 -> xyz=-0.10545 0.33374 -0.05 rpy=-3.1416 0 1.8765
