Commit message: dsdsds

File: 3D_CAD_Scara9/urdf/3D_CAD_Scara9.urdf (robot description, URDF)
Before this commit: robot 3D_CAD_Scara8, 5 links, 4 joints
Links:
- link End_efector_Link: mass 3.121 -> 2.621; geometry collision mesh filename=package://3D_CAD_Scara9/meshes/End_efector_Link.STL; visual mesh filename=package://3D_CAD_Scara9/meshes/End_efector_Link.STL
- link Link01_Link: mass 8.88681009624485 -> 6.88681009624485; geometry collision mesh filename=package://3D_CAD_Scara9/meshes/Link01_Link.STL; visual mesh filename=package://3D_CAD_Scara9/meshes/Link01_Link.STL
- link Link02_Link: geometry collision mesh filename=package://3D_CAD_Scara9/meshes/Link02_Link.STL; visual mesh filename=package://3D_CAD_Scara9/meshes/Link02_Link.STL
- link Link03_Link: mass 3.121 -> 2.621; geometry collision mesh filename=package://3D_CAD_Scara9/meshes/Link03_Link.STL; visual mesh filename=package://3D_CAD_Scara9/meshes/Link03_Link.STL
- link base_link: mass 7.81592864600267 -> 6.24513231920778; geometry collision mesh filename=package://3D_CAD_Scara9/meshes/base_link.STL; visual mesh filename=package://3D_CAD_Scara9/meshes/base_link.STL
Joints:
- joint Endefector_joint: origin xyz=0 0 0.10439 rpy=0 0 0 -> xyz=0 0 0.1 rpy=0 0 0
- joint Joint01_joint: origin xyz=0 0 0.22 rpy=0 0 0 -> xyz=0 0 0.17 rpy=0 0 0
- joint joint02_joint: origin xyz=0.55 0 0.100000000000002 rpy=0 0 0 -> xyz=0.35 0 0.1 rpy=0 0 0
- joint joint03_joint: axis 0 0 1 -> 0 0 -1; limit lower=0 upper=0.20561 effort=0 velocity=0 -> lower=0 upper=0.13 effort=0 velocity=0
