Commit message: kuyyy

File: 3D_CAD_Scara10/urdf/3D_CAD_Scara10.urdf (robot description, URDF)
Before this commit: robot 3D_CAD_Scara9, 5 links, 4 joints
Links:
- link End_efector_Link: geometry collision mesh filename=package://3D_CAD_Scara10/meshes/End_efector_Link.STL; visual mesh filename=package://3D_CAD_Scara10/meshes/End_efector_Link.STL
- link Link01_Link: geometry collision mesh filename=package://3D_CAD_Scara10/meshes/Link01_Link.STL; visual mesh filename=package://3D_CAD_Scara10/meshes/Link01_Link.STL
- link Link02_Link: geometry collision mesh filename=package://3D_CAD_Scara10/meshes/Link02_Link.STL; visual mesh filename=package://3D_CAD_Scara10/meshes/Link02_Link.STL
- link Link03_Link: geometry collision mesh filename=package://3D_CAD_Scara10/meshes/Link03_Link.STL; visual mesh filename=package://3D_CAD_Scara10/meshes/Link03_Link.STL
- link base_link: geometry collision mesh filename=package://3D_CAD_Scara10/meshes/base_link.STL; visual mesh filename=package://3D_CAD_Scara10/meshes/base_link.STL
Joints:
- joint Endefector_joint: origin xyz=0 0 0.1 rpy=0 0 0 -> xyz=0 0 0.0999999999999999 rpy=0 0 0
- joint joint03_joint: axis 0 0 -1 -> 0 0 1; limit lower=0 upper=0.13 effort=0 velocity=0 -> lower=0 upper=0.159999999999085 effort=0 velocity=0; origin xyz=0.35 0.00012531 0.05 rpy=3.1416 0 0 -> xyz=0.35 0.000125314072334626 0.05 rpy=3.14159265358979 0 0
